Commit message: Added materials for running robot in simulation

File: spidar300/sim/urdf/robot.urdf (robot description, URDF)
Before this commit: robot robot, 19 links, 18 joints
Links:
- link Leg_1_: mass None -> 0.0442; geometry collision mesh filename=meshes/collision/Leg_1__0.stl; collision mesh filename=meshes/collision/Leg_1__1.stl
- link Leg_1_coxa: mass None -> 0.1912; geometry collision mesh filename=meshes/collision/Leg_1_coxa_0.stl; collision mesh filename=meshes/collision/Leg_1_coxa_1.stl
- link Leg_1_tibia: mass None -> 0.1596; geometry collision mesh filename=meshes/collision/Leg_1_tibia_0.stl; collision mesh filename=meshes/collision/Leg_1_tibia_1.stl
- link Leg_2_coxa: mass None -> 0.1912; geometry collision mesh filename=meshes/collision/Leg_2_coxa_0.stl; collision mesh filename=meshes/collision/Leg_2_coxa_1.stl
- link Leg_2_femur: mass None -> 0.0442; geometry collision mesh filename=meshes/collision/Leg_2_femur_0.stl; collision mesh filename=meshes/collision/Leg_2_femur_1.stl
- link Leg_2_tibia: mass None -> 0.1596; geometry collision mesh filename=meshes/collision/Leg_2_tibia_0.stl; collision mesh filename=meshes/collision/Leg_2_tibia_1.stl
- link Leg_3_coxa: mass None -> 0.1912; geometry collision mesh filename=meshes/collision/Leg_3_coxa_0.stl; collision mesh filename=meshes/collision/Leg_3_coxa_1.stl
- link Leg_3_femur: mass None -> 0.0442; geometry collision mesh filename=meshes/collision/Leg_3_femur_0.stl; collision mesh filename=meshes/collision/Leg_3_femur_1.stl
- link Leg_3_tibia: mass None -> 0.1595; geometry collision mesh filename=meshes/collision/Leg_3_tibia_0.stl; collision mesh filename=meshes/collision/Leg_3_tibia_1.stl
- link Leg_4_coxa: mass None -> 0.1912; geometry collision mesh filename=meshes/collision/Leg_4_coxa_0.stl; collision mesh filename=meshes/collision/Leg_4_coxa_1.stl
- link Leg_4_femur: mass None -> 0.0442; geometry collision mesh filename=meshes/collision/Leg_4_femur_0.stl; collision mesh filename=meshes/collision/Leg_4_femur_1.stl
- link Leg_4_tibia: mass None -> 0.1596; geometry collision mesh filename=meshes/collision/Leg_4_tibia_0.stl; collision mesh filename=meshes/collision/Leg_4_tibia_1.stl
- link Leg_5_coxa: mass None -> 0.1912; geometry collision mesh filename=meshes/collision/Leg_5_coxa_0.stl; collision mesh filename=meshes/collision/Leg_5_coxa_1.stl
- link Leg_5_femur: mass None -> 0.0442; geometry collision mesh filename=meshes/collision/Leg_5_femur_0.stl; collision mesh filename=meshes/collision/Leg_5_femur_1.stl
- link Leg_5_tibia: mass None -> 0.1596; geometry collision mesh filename=meshes/collision/Leg_5_tibia_0.stl; collision mesh filename=meshes/collision/Leg_5_tibia_1.stl
- link Leg_6_coxa: mass None -> 0.1912; geometry collision mesh filename=meshes/collision/Leg_6_coxa_0.stl; collision mesh filename=meshes/collision/Leg_6_coxa_1.stl
- link Leg_6_femur: mass None -> 0.0442; geometry collision mesh filename=meshes/collision/Leg_6_femur_0.stl; collision mesh filename=meshes/collision/Leg_6_femur_1.stl
- link Leg_6_tibia: mass None -> 0.1596; geometry collision mesh filename=meshes/collision/Leg_6_tibia_0.stl; collision mesh filename=meshes/collision/Leg_6_tibia_1.stl
- link base_link: mass None -> 0.4197; geometry collision mesh filename=meshes/collision/base_link_0.stl; visual mesh filename=meshes/base_link.stl
Joints:
- joint Leg_1_coxa_joint: limit lower=-3.14159 upper=3.14159 effort=10 velocity=1 -> lower=-3.14159 upper=3.14159 effort=1.86 velocity=5.8
- joint Leg_1_femur_joint: limit lower=-3.14159 upper=3.14159 effort=10 velocity=1 -> lower=-3.14159 upper=3.14159 effort=1.86 velocity=5.8
- joint Leg_1_tibia_joint: limit lower=-3.14159 upper=3.14159 effort=10 velocity=1 -> lower=-3.14159 upper=3.14159 effort=1.86 velocity=5.8
- joint Leg_2_coxa_joint: limit lower=-3.14159 upper=3.14159 effort=10 velocity=1 -> lower=-3.14159 upper=3.14159 effort=1.86 velocity=5.8
- joint Leg_2_femur_joint: limit lower=-3.14159 upper=3.14159 effort=10 velocity=1 -> lower=-3.14159 upper=3.14159 effort=1.86 velocity=5.8
- joint Leg_2_tibia_joint: limit lower=-3.14159 upper=3.14159 effort=10 velocity=1 -> lower=-3.14159 upper=3.14159 effort=1.86 velocity=5.8
- joint Leg_3_coxa_joint: limit lower=-3.14159 upper=3.14159 effort=10 velocity=1 -> lower=-3.14159 upper=3.14159 effort=1.86 velocity=5.8
- joint Leg_3_femur_joint: limit lower=-3.14159 upper=3.14159 effort=10 velocity=1 -> lower=-3.14159 upper=3.14159 effort=1.86 velocity=5.8
- joint Leg_3_tibia_joint: limit lower=-3.14159 upper=3.14159 effort=10 velocity=1 -> lower=-3.14159 upper=3.14159 effort=1.86 velocity=5.8
- joint Leg_4_coxa_joint: limit lower=-3.14159 upper=3.14159 effort=10 velocity=1 -> lower=-3.14159 upper=3.14159 effort=1.86 velocity=5.8
- joint Leg_4_femur_joint: limit lower=-3.14159 upper=3.14159 effort=10 velocity=1 -> lower=-3.14159 upper=3.14159 effort=1.86 velocity=5.8
- joint Leg_4_tibia_joint: limit lower=-3.14159 upper=3.14159 effort=10 velocity=1 -> lower=-3.14159 upper=3.14159 effort=1.86 velocity=5.8
- joint Leg_5_coxa_joint: limit lower=-3.14159 upper=3.14159 effort=10 velocity=1 -> lower=-3.14159 upper=3.14159 effort=1.86 velocity=5.8
- joint Leg_5_femur_joint: limit lower=-3.14159 upper=3.14159 effort=10 velocity=1 -> lower=-3.14159 upper=3.14159 effort=1.86 velocity=5.8
- joint Leg_5_tibia_joint: limit lower=-3.14159 upper=3.14159 effort=10 velocity=1 -> lower=-3.14159 upper=3.14159 effort=1.86 velocity=5.8
- joint Leg_6_coxa_joint: limit lower=-3.14159 upper=3.14159 effort=10 velocity=1 -> lower=-3.14159 upper=3.14159 effort=1.86 velocity=5.8
- joint Leg_6_femur_joint: limit lower=-3.14159 upper=3.14159 effort=10 velocity=1 -> lower=-3.14159 upper=3.14159 effort=1.86 velocity=5.8
- joint Leg_6_tibia_joint: limit lower=-3.14159 upper=3.14159 effort=10 velocity=1 -> lower=-3.14159 upper=3.14159 effort=1.86 velocity=5.8

Commit message: Reworked the simulation spider

File: spidar300/sim/urdf/robot.urdf (robot description, URDF)
Before this commit: robot robot, 19 links, 18 joints
Links:
- removed link Leg_1_
- added link Leg_1_femur, mass 0.0442; collision mesh filename=/workspace/code/SO_SPIDAR300/spidar300/sim/urdf/meshes/coll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; collision mesh filename=/workspace/code/SO_SPIDAR300/spidar300/sim/urdf/meshes/coll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
- link Leg_1_coxa: geometry collision mesh filename=/workspace/code/SO_SPIDAR300/spidar300/sim/urdf/meshes/coll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; collision mesh filename=/workspace/code/SO_SPIDAR300/spidar300/sim/urdf/meshes/coll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
- link Leg_1_tibia: geometry collision mesh filename=/workspace/code/SO_SPIDAR300/spidar300/sim/urdf/meshes/coll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; collision mesh filename=/workspace/code/SO_SPIDAR300/spidar300/sim/urdf/meshes/coll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
- link Leg_2_coxa: geometry collision mesh filename=/workspace/code/SO_SPIDAR300/spidar300/sim/urdf/meshes/coll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; collision mesh filename=/workspace/code/SO_SPIDAR300/spidar300/sim/urdf/meshes/coll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
- link Leg_2_femur: geometry collision mesh filename=/workspace/code/SO_SPIDAR300/spidar300/sim/urdf/meshes/coll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; collision mesh filename=/workspace/code/SO_SPIDAR300/spidar300/sim/urdf/meshes/coll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
- link Leg_2_tibia: geometry collision mesh filename=/workspace/code/SO_SPIDAR300/spidar300/sim/urdf/meshes/coll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; collision mesh filename=/workspace/code/SO_SPIDAR300/spidar300/sim/urdf/meshes/coll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
- link Leg_3_coxa: geometry collision mesh filename=/workspace/code/SO_SPIDAR300/spidar300/sim/urdf/meshes/coll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; collision mesh filename=/workspace/code/SO_SPIDAR300/spidar300/sim/urdf/meshes/coll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
- link Leg_3_femur: geometry collision mesh filename=/workspace/code/SO_SPIDAR300/spidar300/sim/urdf/meshes/coll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; collision mesh filename=/workspace/code/SO_SPIDAR300/spidar300/sim/urdf/meshes/coll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
- link Leg_3_tibia: geometry collision mesh filename=/workspace/code/SO_SPIDAR300/spidar300/sim/urdf/meshes/coll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; collision mesh filename=/workspace/code/SO_SPIDAR300/spidar300/sim/urdf/meshes/coll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
- link Leg_4_coxa: geometry collision mesh filename=/workspace/code/SO_SPIDAR300/spidar300/sim/urdf/meshes/coll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; collision mesh filename=/workspace/code/SO_SPIDAR300/spidar300/sim/urdf/meshes/coll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
- link Leg_4_femur: geometry collision mesh filename=/workspace/code/SO_SPIDAR300/spidar300/sim/urdf/meshes/coll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; collision mesh filename=/workspace/code/SO_SPIDAR300/spidar300/sim/urdf/meshes/coll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
- link Leg_4_tibia: geometry collision mesh filename=/workspace/code/SO_SPIDAR300/spidar300/sim/urdf/meshes/coll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; collision mesh filename=/workspace/code/SO_SPIDAR300/spidar300/sim/urdf/meshes/coll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
- link Leg_5_coxa: geometry collision mesh filename=/workspace/code/SO_SPIDAR300/spidar300/sim/urdf/meshes/coll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; collision mesh filename=/workspace/code/SO_SPIDAR300/spidar300/sim/urdf/meshes/coll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
- link Leg_5_femur: geometry collision mesh filename=/workspace/code/SO_SPIDAR300/spidar300/sim/urdf/meshes/coll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; collision mesh filename=/workspace/code/SO_SPIDAR300/spidar300/sim/urdf/meshes/coll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
- link Leg_5_tibia: geometry collision mesh filename=/workspace/code/SO_SPIDAR300/spidar300/sim/urdf/meshes/coll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; collision mesh filename=/workspace/code/SO_SPIDAR300/spidar300/sim/urdf/meshes/coll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
- link Leg_6_coxa: geometry collision mesh filename=/workspace/code/SO_SPIDAR300/spidar300/sim/urdf/meshes/coll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; collision mesh filename=/workspace/code/SO_SPIDAR300/spidar300/sim/urdf/meshes/coll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
- link Leg_6_femur: geometry collision mesh filename=/workspace/code/SO_SPIDAR300/spidar300/sim/urdf/meshes/coll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; collision mesh filename=/workspace/code/SO_SPIDAR300/spidar300/sim/urdf/meshes/coll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
- link Leg_6_tibia: geometry collision mesh filename=/workspace/code/SO_SPIDAR300/spidar300/sim/urdf/meshes/coll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; collision mesh filename=/workspace/code/SO_SPIDAR300/spidar300/sim/urdf/meshes/coll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
- link base_link: geometry collision mesh filename=/workspace/code/SO_SPIDAR300/spidar300/sim/urdf/meshes/coll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; visual mesh filename=/workspace/code/SO_SPIDAR300/spidar300/sim/urdf/meshes/base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
Joints:
- joint Leg_1_coxa_joint: limit lower=-3.14159 upper=3.14159 effort=1.86 velocity=5.8 -> lower=-1.45 upper=1.508 effort=1.9 velocity=4.7
- joint Leg_1_femur_joint: child Leg_1_ -> Leg_1_femur; limit lower=-3.14159 upper=3.14159 effort=1.86 velocity=5.8 -> lower=-2.2 upper=2.5 effort=1.9 velocity=4.7
- joint Leg_1_tibia_joint: limit lower=-3.14159 upper=3.14159 effort=1.86 velocity=5.8 -> lower=-1.477 upper=1.66 effort=1.9 velocity=4.7; parent Leg_1_ -> Leg_1_femur
- joint Leg_2_coxa_joint: limit lower=-3.14159 upper=3.14159 effort=1.86 velocity=5.8 -> lower=-1.45 upper=1.508 effort=1.9 velocity=4.7
- joint Leg_2_femur_joint: limit lower=-3.14159 upper=3.14159 effort=1.86 velocity=5.8 -> lower=-2.2 upper=2.5 effort=1.9 velocity=4.7
- joint Leg_2_tibia_joint: limit lower=-3.14159 upper=3.14159 effort=1.86 velocity=5.8 -> lower=-1.477 upper=1.66 effort=1.9 velocity=4.7
- joint Leg_3_coxa_joint: limit lower=-3.14159 upper=3.14159 effort=1.86 velocity=5.8 -> lower=-1.45 upper=1.508 effort=1.9 velocity=4.7
- joint Leg_3_femur_joint: limit lower=-3.14159 upper=3.14159 effort=1.86 velocity=5.8 -> lower=-2.2 upper=2.5 effort=1.9 velocity=4.7
- joint Leg_3_tibia_joint: limit lower=-3.14159 upper=3.14159 effort=1.86 velocity=5.8 -> lower=-1.477 upper=1.66 effort=1.9 velocity=4.7
- joint Leg_4_coxa_joint: limit lower=-3.14159 upper=3.14159 effort=1.86 velocity=5.8 -> lower=-1.45 upper=1.508 effort=1.9 velocity=4.7
- joint Leg_4_femur_joint: limit lower=-3.14159 upper=3.14159 effort=1.86 velocity=5.8 -> lower=-2.2 upper=2.5 effort=1.9 velocity=4.7
- joint Leg_4_tibia_joint: limit lower=-3.14159 upper=3.14159 effort=1.86 velocity=5.8 -> lower=-1.477 upper=1.66 effort=1.9 velocity=4.7
- joint Leg_5_coxa_joint: limit lower=-3.14159 upper=3.14159 effort=1.86 velocity=5.8 -> lower=-1.45 upper=1.508 effort=1.9 velocity=4.7
- joint Leg_5_femur_joint: limit lower=-3.14159 upper=3.14159 effort=1.86 velocity=5.8 -> lower=-2.2 upper=2.5 effort=1.9 velocity=4.7
- joint Leg_5_tibia_joint: limit lower=-3.14159 upper=3.14159 effort=1.86 velocity=5.8 -> lower=-1.477 upper=1.66 effort=1.9 velocity=4.7
- joint Leg_6_coxa_joint: limit lower=-3.14159 upper=3.14159 effort=1.86 velocity=5.8 -> lower=-1.45 upper=1.508 effort=1.9 velocity=4.7
- joint Leg_6_femur_joint: limit lower=-3.14159 upper=3.14159 effort=1.86 velocity=5.8 -> lower=-2.2 upper=2.5 effort=1.9 velocity=4.7
- joint Leg_6_tibia_joint: limit lower=-3.14159 upper=3.14159 effort=1.86 velocity=5.8 -> lower=-1.477 upper=1.66 effort=1.9 velocity=4.7
